File: Lion1.brd (EAGLE design)
At the start: 100 x 85.7 mm, 62 parts, among them IC1 MCP4822, IC2 MCP4822, IC3 MCP4822, IC4 REG1117, U7 2564-, U8 2564-

Commit message: no message
Parts:
- added C15: 4.7uf, rcl:C050-025X075
- added C16, C17, C18, C19: 4.7uF, rcl:C050-025X075
- added C20: 100nf, rcl:C0805
- added JP15: AUX, pinhead:1X04
- added R26, R27: 1K, SmartPrj:0204/7
- C12: value (none) -> 47uf; device rc-master:CE-025X065 -> rc-master:CE-025X060
- C13, C5, C7: value (none) -> 100nf
- C14: value (none) -> 100uf; device rc-master:CE-025X065 -> rc-master:CE-025X060
- C3: value (none) -> 100pf
- C8: value (none) -> 22uf; device rc-master:CE-025X065 -> rc-master:CE-025X060
- R10: value (none) -> 1K
- R11: value (none) -> 2K
- R12: value (none) -> 75 Ohm
- R13: value (none) -> 100 Ohm
- R15, R16, R17, R18: device SmartPrj:0204/7 -> SmartPrj:0204V
- R20, R21: value (none) -> 100
- R25: value (none) -> 4.7K
- R9: value (none) -> 500 Ohm
- moved R18 5.24 mm to (57.1, 28.6)
- moved R17 5.12 mm to (60.3, 28.6)
- moved R16 5.12 mm to (66.7, 28.6)
- moved R15 5.08 mm to (63.5, 28.6)
- moved U$1 2.01 mm to (49.5, 24.8)
- moved R23 2.01 mm to (54.0, 38.7)
- moved C5 2.01 mm to (74.9, 43.2)
- moved C7 1.42 mm to (29.2, 34.9)
- moved C8 1.27 mm to (43.8, 33.7)
- moved C10 1.27 mm to (42.5, 25.4)
- moved IC1 1.27 mm to (63.5, 36.8)
- moved R19 0.90 mm to (52.7, 32.4)
- moved C11 0.90 mm to (55.2, 45.1), turned to 180 degrees
- moved R24 0.90 mm to (56.5, 38.7)
- moved C6 0.90 mm to (64.8, 45.1)
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Connections:
- removed net N$16: U7.35
- new net N$21: C16.2, R16.1
- new net N$22: C17.2, R17.1
- new net N$23: C18.2, R18.1
- new net N$24: JP15.2, U7.35
- new net N$3: C19.2, R26.2, R27.1, U$1.3, U$1.5
- new net N$4: C15.2, R15.1
- net 3V3: now also C20.2; no longer C10.2
- net 5V: now also C10.2, R27.2
- net AUDIOA: now also C15.1; no longer R15.1
- net AUDIOB: now also C16.1; no longer R16.1
- net AUDIOC: now also C17.1; no longer R17.1
- net GND: now also C19.1, C20.1, R26.1; no longer U$1.3, U$1.5
- net N$85: now also JP15.3
- net NOISEO: now also C18.1; no longer R18.1
Routing:
- net 5V: track 81.9 -> 125.2 mm, vias 0 -> 1
- net A16: track 55.7 -> 97.2 mm
- net GND: track 517.6 -> 559.1 mm
- net INT: track 27.4 -> 60.2 mm
- net A2: track 64.7 -> 33.9 mm
- net N$3: track 0.00 -> 25.3 mm
- net ER_SEL: track 59.7 -> 37.7 mm, vias 0 -> 1
- net 3V3: track 169.4 -> 148.1 mm, vias 2 -> 4
- net HOLD: track 17.0 -> 34.4 mm
- net D1: track 45.9 -> 63.3 mm
- net SPICS2: track 63.9 -> 80.6 mm, vias 0 -> 1
- net D3: track 45.2 -> 60.9 mm, vias 1 -> 2
- net JOY2[1]: track 26.5 -> 12.0 mm
- net N$13: track 32.8 -> 46.8 mm
- net VSYN2: track 39.5 -> 25.8 mm
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