File: Lion1.sch (EAGLE design)
At the start: 62 parts, among them IC1 MCP4822, IC2 MCP4822, IC3 MCP4822, IC4 REG1117, U7 2564-, U8 2564-

Commit message: no message
Parts:
- added C15: 4.7uf, rcl:C-EU050-025X075
- added C16, C17, C18, C19: 4.7uF, rcl:C-EU050-025X075
- added C20: 100nf, rcl:C-EUC0805
- added JP15: AUX, pinhead:PINHD-1X4
- added R26, R27: 1K, SmartPrj:R-EU_0204/7
- C12: value (none) -> 47uf; device rc-master:CP_E-025X065 -> rc-master:CP_E-025X060
- C13, C5, C7: value (none) -> 100nf
- C14: value (none) -> 100uf; device rc-master:CP_E-025X065 -> rc-master:CP_E-025X060
- C3: value (none) -> 100pf
- C8: value (none) -> 22uf; device rc-master:CP_E-025X065 -> rc-master:CP_E-025X060
- R10: value (none) -> 1K
- R11: value (none) -> 2K
- R12: value (none) -> 75 Ohm
- R13: value (none) -> 100 Ohm
- R15, R16, R17, R18: device SmartPrj:R-EU_0204/7 -> SmartPrj:R-EU_0204/2V
- R20, R21: value (none) -> 100
- R25: value (none) -> 4.7K
- R9: value (none) -> 500 Ohm
Connections:
- removed net N$16: U7-35.KL
- new net N$21: C16.2, R16.1
- new net N$22: C17.2, R17.1
- new net N$23: C18.2, R18.1
- new net N$24: JP15.2, U7-35.KL
- new net N$3: C19.2, R26.2, R27.1, U$1A.+IN, U$1B.+IN
- new net N$4: C15.2, R15.1
- net 3V3: now also C20.2; no longer C10.2
- net 5V: now also C10.2, R27.2
- net AUDIOA: now also C15.1; no longer R15.1
- net AUDIOB: now also C16.1; no longer R16.1
- net AUDIOC: now also C17.1; no longer R17.1
- net GND: now also C19.1, C20.1, R26.1; no longer U$1A.+IN, U$1B.+IN
- net N$85: now also JP15.3
- net NOISEO: now also C18.1; no longer R18.1
Other:
- moved on the sheet: C10, R1, R11, R15, R16, R17, R18, R3, R5, R7, R9
