File: Lion1_2.sch (EAGLE design)
At the start: 71 parts, among them IC1 MCP4822, IC2 MCP4822, IC3 MCP4822, IC4 REG1117, U7 2564-, U8 2564-

Commit message: v2
Parts:
- removed JP14: (no value), pinhead:PINHD-1X1
- added C21, C22: 4.7uf, rcl:C-EU050-025X075
- added R28, R29: (no value), SmartPrj:R-EU_0204/2V
- C13: value 100nf -> (none)
Connections:
- net N$24 renamed TX2
- net N$85 renamed RX2
- removed net 3V3: C20.2, C7.2, JP1.4, JP10.2, JP10.4, JP10.6, R25.2, U$2G$2.VCC, U$2G$3.VCC, U7-3.KL, U7-4.KL, U8-3.KL, U8-4.KL
- removed net GND: C1.1, C10.1, C11.2, C12.-, C13.1, C14.-, C19.1, C2.1, C20.1, C3.1, C4.1, C5.1, C6.1, C7.1, C9.1, IC1P.GND, IC2P.GND, IC3P.GND, IC4.GND, JP1.1, JP11.1, JP12.1, JP13.1, JP2.4, JP3.2, JP4.2, JP5.2, JP6.2, JP7.4, JP8.4, JP9.2, R12.1, R26.1, R4.1, R8.1, U$1P.V-, U$2G$4.VSS, U$2G$5.VSS, U7-1.KL, U7-2.KL, U7-5.KL, U7-6.KL, U7-61.KL, U7-62.KL, U8-1.KL, U8-2.KL, U8-5.KL, U8-6.KL, U8-61.KL, U8-62.KL, VGA1G$1.GND@0, VGA1G$1.GND@1
- removed net N$70: U8-64.KL
- new net 3V3_7: C20.2, C7.2, JP15.1, U$2G$2.VCC, U$2G$3.VCC, U7-3.KL, U7-4.KL
- new net 3V3_8: JP1.4, JP10.2, JP10.4, JP10.6, R25.2, U8-3.KL, U8-4.KL
- new net ADD: C21.1, C22.1, R15.2, R16.2, R17.2, R18.2, R19.1, U$1A.-IN
- new net GND7_61: C1.1, C2.1, C3.1, JP15.4, JP2.4, R12.1, R4.1, R8.1, U7-61.KL, U7-62.KL, VGA1G$1.GND@0, VGA1G$1.GND@1
- new net GND8_1: C10.1, C11.2, C19.1, JP1.1, JP13.1, JP6.2, JP7.4, JP9.2, R26.1, U$1P.V-, U8-1.KL, U8-2.KL, U8-5.KL, U8-6.KL
- new net GND_: C12.-, C13.1, C14.-, C4.1, C5.1, C6.1, C9.1, IC1P.GND, IC2P.GND, IC3P.GND, IC4.GND, JP12.1, JP3.2, JP4.2, JP5.2, JP8.4, U8-61.KL, U8-62.KL
- new net GND_1: C20.1, C7.1, JP11.1, U$2G$4.VSS, U$2G$5.VSS, U7-1.KL, U7-2.KL, U7-5.KL, U7-6.KL
- new net N$25: C22.2, R29.1
- new net N$26: IC1A.VOUTB, R29.2
- net 5V: now also U8-64.KL
- net 5V_2: now also U7-64.KL
- net N$2: now also R28.2; no longer JP14.1
- net N$9: now also C21.2, R28.1; no longer R15.2, R16.2, R17.2, R18.2, R19.1, U$1A.-IN
Other:
- moved on the sheet: C11
